File: stm32_tx/emi_filter.kicad_sch (KiCad schematic)
At the start: 16 parts, among them J3 IEC_60320_C14_Receptacle

Commit message: Updated file paths in TX project
Parts:
- C47: value 2u2, X2, 305Vac -> 2u2, X2, 305Vac, MXT225K305H23
- C49, C50: value 2.2uF, X2, 305Vac -> 2.2uF, X2, 305Vac, MXT225K305H23
- C53: value NM, X2, 305Vac -> NM, X2, 305Vac, MXT225K305H23
- F1: value TBD -> 15A
Changed lines of the file:
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@@
 			)
 		)
-		(property "Value" "2.2uF, X2, 305Vac"
+		(property "Value" "2.2uF, X2, 305Vac, MXT225K305H23"
 			(at 144.018 99.568 0)
 			(effects
@@
 			)
 		)
-		(property "Value" "NM, X2, 305Vac"
+		(property "Value" "NM, X2, 305Vac, MXT225K305H23"
 			(at 231.14 97.7899 0)
 			(effects
@@
 		)
 		(property "Value" "MOV-14D561K"
-			(at 212.344 102.362 0)
+			(at 213.106 91.948 0)
 			(effects
 				(font
@@
 		(on_board yes)
 		(dnp no)
-		(fields_autoplaced yes)
 		(property "Reference" "C47"
-			(at 83.82 91.4399 0)
-			(effects
-				(font
-					(size 1.27 1.27)
-				)
-				(justify left)
-			)
-		)
-		(property "Value" "2u2, X2, 305Vac"
-			(at 83.82 93.9799 0)
+			(at 81.788 96.012 0)
+			(effects
+				(font
+					(size 1.27 1.27)
+				)
+				(justify left)
+			)
+		)
+		(property "Value" "2u2, X2, 305Vac, MXT225K305H23"
+			(at 83.566 99.822 0)
 			(effects
 				(font
@@
 			)
 		)
-		(property "Value" "2.2uF, X2, 305Vac"
-			(at 191.516 101.6 0)
+		(property "Value" "2.2uF, X2, 305Vac, MXT225K305H23"
+			(at 180.594 104.394 0)
 			(effects
 				(font
@@
 			)
 		)
-		(property "Value" "TBD"
+		(property "Value" "15A"
 			(at 57.15 67.31 90)
 			(effects
