File: stm32_tx/High_voltage_auxiliary.kicad_sch (KiCad schematic)
At the start: 2 parts, among them U10 RP-1212S, U4 IRM-01-3.3

Commit message: Added selected footprints
Parts:
- U10: footprint RP_S_RCP -> WPT_TX:RP_S_RCP
- U4: footprint IRM02_MWU -> WPT_TX:IRM02_MWU
Changed lines of the file:
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@@
 			)
 		)
-		(property "Footprint" "RP_S_RCP"
+		(property "Footprint" "WPT_TX:RP_S_RCP"
 			(at 208.28 142.24 0)
 			(effects
@@
 			)
 		)
-		(property "Footprint" "IRM02_MWU"
+		(property "Footprint" "WPT_TX:IRM02_MWU"
 			(at 209.55 119.38 0)
 			(effects
