File: stm32_tx/high_voltage_inverter.kicad_sch (KiCad schematic)
At the start: 15 parts, among them U5 IPW65R041CFD7XKSA1, U6 IPW65R041CFD7XKSA1, U7 IPW65R041CFD7XKSA1, U8 IPW65R041CFD7XKSA1

Commit message: Added components and structure for analogue overvoltage and overcurrent protection
Parts:
- added R20: 50 ohm, 100W, symbol Device:R
- added U19: IPW65R041CFD7XKSA1, WPT_TX:PG-TO247-3-41, symbol IPW65r04:IPW65R041CFD7XKSA1
- C132: renamed from C_TX_COMP; value 250n -> 250nF
- renumbered LL_TX to L143
Connections:
- net +325V: now also R20.2
- net GND_HV: now also U19.3 (SOURCE)
- new net: R20.1, U19.2 (DRAIN)
- new net OVP: U19.1 (GATE)
Other:
- moved on the sheet: C11, C132, D2, D4, D7, D8, L143, R12, R13, R14, R15, U5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

Commit message: Added selected footprints
Parts:
- C11: footprint (none) -> Capacitor_SMD:C_0805_2012Metric
- C132: footprint (none) -> Capacitor_SMD:C_0402_1005Metric
- R12, R13, R14, R15: footprint (none) -> Resistor_SMD:R_1206_3216Metric
- U6, U7, U8: footprint PG-TO247-3-41 -> WPT_TX:PG-TO247-3-41
Changed lines of the file:
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@@
 			)
 		)
-		(property "Footprint" "PG-TO247-3-41"
+		(property "Footprint" "WPT_TX:PG-TO247-3-41"
 			(at 125.73 113.03 0)
 			(effects
@@
 			)
 		)
-		(property "Footprint" ""
+		(property "Footprint" "Capacitor_SMD:C_0402_1005Metric"
 			(at 255.27 93.0148 0)
 			(effects
@@
 			)
 		)
-		(property "Footprint" ""
+		(property "Footprint" "Resistor_SMD:R_1206_3216Metric"
 			(at 119.38 114.808 90)
 			(effects
@@
 			)
 		)
-		(property "Footprint" "PG-TO247-3-41"
+		(property "Footprint" "WPT_TX:PG-TO247-3-41"
 			(at 193.04 67.31 0)
 			(effects
@@
 			)
 		)
-		(property "Footprint" ""
+		(property "Footprint" "Resistor_SMD:R_1206_3216Metric"
 			(at 119.38 70.358 90)
 			(effects
@@
 			)
 		)
-		(property "Footprint" ""
+		(property "Footprint" "Resistor_SMD:R_1206_3216Metric"
 			(at 186.69 69.088 90)
 			(effects
@@
 			)
 		)
-		(property "Footprint" "PG-TO247-3-41"
+		(property "Footprint" "WPT_TX:PG-TO247-3-41"
 			(at 193.04 114.3 0)
 			(effects
@@
 			)
 		)
-		(property "Footprint" ""
+		(property "Footprint" "Capacitor_SMD:C_0805_2012Metric"
 			(at 33.9852 99.06 0)
 			(effects
@@
 			)
 		)
-		(property "Footprint" ""
+		(property "Footprint" "Resistor_SMD:R_1206_3216Metric"
 			(at 186.69 116.078 90)
 			(effects
