File: stm32_tx/low_voltage_5V_buck.kicad_sch (KiCad schematic)
At the start: 8 parts, among them U12 TPS5430DDA

Commit message: Added selected footprints
Parts:
- C7: footprint (none) -> Capacitor_SMD:C_0402_1005Metric
Changed lines of the file:
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@@
 			)
 		)
-		(property "Footprint" ""
+		(property "Footprint" "Capacitor_SMD:C_0402_1005Metric"
 			(at 143.51 77.7748 0)
 			(effects
