File: stm32_tx/stm_MCU.kicad_sch (KiCad schematic)
At the start: 17 parts, among them J2 Conn_01x04_Pin, SW1 SW_SPDT, SW2 SW_MEC_5G, U1 STM32G071CBT6, U2 AMS1117-3.3, Y1 Crystal1

Commit message: Added selected footprints
Parts:
- C1, C2, C3, C4: footprint (none) -> Capacitor_SMD:C_0402_1005Metric
Changed lines of the file:
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@@
 			)
 		)
-		(property "Footprint" ""
+		(property "Footprint" "Capacitor_SMD:C_0402_1005Metric"
 			(at 261.3152 86.36 0)
 			(effects
@@
 			)
 		)
-		(property "Footprint" ""
+		(property "Footprint" "Capacitor_SMD:C_0402_1005Metric"
 			(at 275.2852 86.36 0)
 			(effects
@@
 			)
 		)
-		(property "Footprint" ""
+		(property "Footprint" "Capacitor_SMD:C_0402_1005Metric"
 			(at 195.2752 68.58 0)
 			(effects
@@
 			)
 		)
-		(property "Footprint" ""
+		(property "Footprint" "Capacitor_SMD:C_0402_1005Metric"
 			(at 202.8952 68.58 0)
 			(effects
