File: stm32_rx/high_voltage.kicad_sch (KiCad schematic)
At the start: 12 parts

Commit message: Updated file paths in TX project
Parts:
- removed C1: 250n, symbol Device:C
- removed C54: 470uF, symbol Device:C
- removed CR1, CR2, CR3, CR5: STPSC10H065B-TR, WPT_TX:DPAK_STPS_STM, symbol 2026-07-24_14-19-21:STPSC10H065B-TR
- removed LL_TX: 70uH, 35Khz, symbol Device:L_Ferrite
- removed R1: 0.5, symbol Device:R
- removed RBleed1, RBleed2, RBleed3, RBleed4: 22k, symbol Device:R
Connections:
- no-connect marks 4 -> 0
Other:
- added sheet High Voltage ADC (high_voltage_adc.kicad_sch)
- added sheet rectifier (high_voltage_rectifier.kicad_sch)

Commit message: I can't find the right module
Parts:
- added PS1: PXC-M10-24WD05, PXC-M10-24WD05:CONV_PXC-M10-24WD05, symbol PXC-M10-24WD05:PXC-M10-24WD05
- added U10: RP-1212S, WPT_TX:RP_S_RCP, symbol 2026-09-17_07-04-30:RP-1212S
Connections:
- new net +12V_HV: PS1.14 (+VOUT), U10.1 (+VIN)
- new net +12V_LV: U10.7 (+VOUT)
- new net GND_HV: PS1.11 (-VOUT), PS1.2 (-VIN), U10.2 (-VIN)
- new net GND_LV: U10.5 (-VOUT)
- new net V_RX: PS1.22 (+VIN), PS1.23 (+VIN)
